File: Design Files/KIcad Files/Explore Clock.sch (KiCad schematic (older format))
At the start: 24 parts, among them CON1 BARREL_JACK, IC1 ATMEGA328P-P, P1 CONN_01X07, Q1 BC547, Q2 BC547, Q3 IRF540N, SW1 SW_PUSH, SW2 SW_PUSH, U1 LDR, Y1 32.768KHz

Commit message: Layout For pcb and Acrylic Design Uploaded
Parts:
- added U2, U3, U4, U5: MountingHole, symbol MountingHole
- added U6: EE_Logo, symbol EE_Logo
Connections:
- net GND: now also R7.2
Changed lines of the file:
@@
 LIBS:w_opto
 LIBS:led
+LIBS:ExploreM3-cache
+LIBS:ExploreM3
 LIBS:Explore Clock-cache
 EELAYER 25 0
@@
 91 D7 3E FA 04 87 BF 7F D8 87 EE E1 C8 9C A2 F7 E4 7B 47 1A 21 A9 E9 AE A6 61 E6 63 11 EF 34 7D
 BD EE 38 A9 51 41 6E 70 71 54 41 3F EC 42 8E BC AB 3D C0 C1 9B A3 8E FF 0F 71 E1 17 88 11 2B 92
-BC 00 00 00 00 49 45 4E 44 AE 42 60 82 4C
+BC 00 00 00 00 49 45 4E 44 AE 42 60 82 DC
 EndData
 $EndBitmap
@@
 DIY - Explore clock
 $Comp
-L VCC #PWR8
+L VCC #PWR01
 U 1 1 57EF8CD9
 P 6150 1200
-F 0 "#PWR8" H 6150 1050 50  0001 C CNN
+F 0 "#PWR01" H 6150 1050 50  0001 C CNN
 F 1 "VCC" H 6150 1350 50  0000 C CNN
 F 2 "" H 6150 1200 50  0000 C CNN
@@
 $EndComp
 $Comp
-L GND #PWR7
+L GND #PWR02
 U 1 1 57EF8E24
 P 6100 3800
-F 0 "#PWR7" H 6100 3550 50  0001 C CNN
+F 0 "#PWR02" H 6100 3550 50  0001 C CNN
 F 1 "GND" H 6100 3650 50  0000 C CNN
 F 2 "" H 6100 3800 50  0000 C CNN
@@
 $EndComp
 $Comp
-L GND #PWR4
+L GND #PWR03
 U 1 1 57EFA30E
 P 2550 2200
-F 0 "#PWR4" H 2550 1950 50  0001 C CNN
+F 0 "#PWR03" H 2550 1950 50  0001 C CNN
 F 1 "GND" H 2550 2050 50  0000 C CNN
 F 2 "" H 2550 2200 50  0000 C CNN
@@
 $EndComp
 $Comp
-L GND #PWR5
+L GND #PWR04
 U 1 1 57EFA330
 P 2550 3000
-F 0 "#PWR5" H 2550 2750 50  0001 C CNN
+F 0 "#PWR04" H 2550 2750 50  0001 C CNN
 F 1 "GND" H 2550 2850 50  0000 C CNN
 F 2 "" H 2550 3000 50  0000 C CNN
@@
 $EndComp
 $Comp
-L VCC #PWR6
+L VCC #PWR05
 U 1 1 57EFA64B
 P 3500 1450
-F 0 "#PWR6" H 3500 1300 50  0001 C CNN
+F 0 "#PWR05" H 3500 1300 50  0001 C CNN
 F 1 "VCC" H 3500 1600 50  0000 C CNN
 F 2 "" H 3500 1450 50  0000 C CNN
@@
 $EndComp
 $Comp
-L GND #PWR1
+L GND #PWR06
 U 1 1 57EFCEE9
 P 2300 6050
-F 0 "#PWR1" H 2300 5800 50  0001 C CNN
+F 0 "#PWR06" H 2300 5800 50  0001 C CNN
 F 1 "GND" H 2300 5900 50  0000 C CNN
 F 2 "" H 2300 6050 50  0000 C CNN
@@
 NoConn ~ 2050 6400
 $Comp
-L VCC #PWR2
+L VCC #PWR07
 U 1 1 57EFD128
 P 2300 6450
-F 0 "#PWR2" H 2300 6300 50  0001 C CNN
+F 0 "#PWR07" H 2300 6300 50  0001 C CNN
 F 1 "VCC" H 2300 6600 50  0000 C CNN
 F 2 "" H 2300 6450 50  0000 C CNN
@@
 $EndComp
 $Comp
-L GND #PWR15
+L GND #PWR08
 U 1 1 57F098A3
 P 10150 4050
-F 0 "#PWR15" H 10150 3800 50  0001 C CNN
+F 0 "#PWR08" H 10150 3800 50  0001 C CNN
 F 1 "GND" H 10150 3900 50  0000 C CNN
 F 2 "" H 10150 4050 50  0000 C CNN
@@
 $EndComp
 $Comp
-L VCC #PWR14
+L VCC #PWR09
 U 1 1 57F09B6A
 P 10150 2300
-F 0 "#PWR14" H 10150 2150 50  0001 C CNN
+F 0 "#PWR09" H 10150 2150 50  0001 C CNN
 F 1 "VCC" H 10150 2450 50  0000 C CNN
 F 2 "" H 10150 2300 50  0000 C CNN
@@
 $EndComp
 $Comp
-L VCC #PWR16
+L VCC #PWR010
 U 1 1 57F0D12E
 P 10200 4600
-F 0 "#PWR16" H 10200 4450 50  0001 C CNN
+F 0 "#PWR010" H 10200 4450 50  0001 C CNN
 F 1 "VCC" H 10200 4750 50  0000 C CNN
 F 2 "" H 10200 4600 50  0000 C CNN
@@
 $EndComp
 $Comp
-L GND #PWR9
+L GND #PWR011
 U 1 1 57F1136E
 P 8400 5800
-F 0 "#PWR9" H 8400 5550 50  0001 C CNN
+F 0 "#PWR011" H 8400 5550 50  0001 C CNN
 F 1 "GND" H 8400 5650 50  0000 C CNN
 F 2 "" H 8400 5800 50  0000 C CNN
@@
 Micro controller and circuitry
 $Comp
-L VCC #PWR10
+L VCC #PWR012
 U 1 1 57F1B754
 P 9450 2200
-F 0 "#PWR10" H 9450 2050 50  0001 C CNN
+F 0 "#PWR012" H 9450 2050 50  0001 C CNN
 F 1 "VCC" H 9450 2350 50  0000 C CNN
 F 2 "" H 9450 2200 50  0000 C CNN
@@
 	2650 1350 2650 1250
 $Comp
-L GND #PWR3
+L GND #PWR013
 U 1 1 57F34AB2
 P 2350 1000
-F 0 "#PWR3" H 2350 750 50  0001 C CNN
+F 0 "#PWR013" H 2350 750 50  0001 C CNN
 F 1 "GND" H 2350 850 50  0000 C CNN
 F 2 "" H 2350 1000 50  0000 C CNN
@@
 $EndComp
 $Comp
-L VCC #PWR12
+L VCC #PWR014
 U 1 1 57F35B1B
 P 9875 1025
-F 0 "#PWR12" H 9875 875 50  0001 C CNN
+F 0 "#PWR014" H 9875 875 50  0001 C CNN
 F 1 "VCC" H 9875 1175 50  0000 C CNN
 F 2 "" H 9875 1025 50  0000 C CNN
@@
 $EndComp
 $Comp
-L GND #PWR13
+L GND #PWR015
 U 1 1 57F35D0A
 P 9875 2050
-F 0 "#PWR13" H 9875 1800 50  0001 C CNN
+F 0 "#PWR015" H 9875 1800 50  0001 C CNN
 F 1 "GND" H 9875 1900 50  0000 C CNN
 F 2 "" H 9875 2050 50  0000 C CNN
@@
 	1    0    0    -1
 $EndComp
-Wire Wire Line
-	10200 5650 10200 6050
-$Comp
-L GND #PWR11
+$Comp
+L GND #PWR016
 U 1 1 57F3A574
 P 9850 6350
-F 0 "#PWR11" H 9850 6100 50  0001 C CNN
+F 0 "#PWR016" H 9850 6100 50  0001 C CNN
 F 1 "GND" H 9850 6200 50  0000 C CNN
 F 2 "" H 9850 6350 50  0000 C CNN
@@
 Connection ~ 10200 5950
 $Comp
-L GND #PWR17
+L GND #PWR017
 U 1 1 57F3C1E0
-P 10200 6400
-F 0 "#PWR17" H 10200 6150 50  0001 C CNN
-F 1 "GND" H 10350 6300 50  0000 C CNN
-F 2 "" H 10200 6400 50  0000 C CNN
-F 3 "" H 10200 6400 50  0000 C CNN
-	1    10200 6400
-	1    0    0    -1
-$EndComp
-Wire Wire Line
-	10200 6400 10200 6350
+P 10200 6450
+F 0 "#PWR017" H 10200 6200 50  0001 C CNN
+F 1 "GND" H 10350 6350 50  0000 C CNN
+F 2 "" H 10200 6450 50  0000 C CNN
+F 3 "" H 10200 6450 50  0000 C CNN
+	1    10200 6450
+	1    0    0    -1
+$EndComp
 Wire Wire Line
 	9850 5750 9850 5500
@@
 Wire Wire Line
 	8550 2250 8350 2250
+$Comp
+L MountingHole U2
+U 1 1 57F63CCF
+P 925 4725
+F 0 "U2" H 925 4575 40  0000 C CNN
+F 1 "MountingHole" H 925 4625 40  0000 C CNN
+F 2 "" H 925 4725 40  0000 C CNN
+F 3 "" H 925 4725 40  0000 C CNN
+	1    925  4725
+	1    0    0    -1
+$EndComp
+$Comp
+L MountingHole U3
+U 1 1 57F63E2F
+P 1425 4725
+F 0 "U3" H 1425 4575 40  0000 C CNN
+F 1 "MountingHole" H 1425 4625 40  0000 C CNN
+F 2 "" H 1425 4725 40  0000 C CNN
+F 3 "" H 1425 4725 40  0000 C CNN
+	1    1425 4725
+	1    0    0    -1
+$EndComp
+$Comp
+L MountingHole U4
+U 1 1 57F63E83
+P 1925 4725
+F 0 "U4" H 1925 4575 40  0000 C CNN
+F 1 "MountingHole" H 1925 4625 40  0000 C CNN
+F 2 "" H 1925 4725 40  0000 C CNN
+F 3 "" H 1925 4725 40  0000 C CNN
+	1    1925 4725
+	1    0    0    -1
+$EndComp
+$Comp
+L MountingHole U5
+U 1 1 57F63EC8
+P 2450 4725
+F 0 "U5" H 2450 4575 40  0000 C CNN
+F 1 "MountingHole" H 2450 4625 40  0000 C CNN
+F 2 "" H 2450 4725 40  0000 C CNN
+F 3 "" H 2450 4725 40  0000 C CNN
+	1    2450 4725
+	1    0    0    -1
+$EndComp
+$Comp
+L EE_Logo U6
+U 1 1 57F643BB
+P 925 5175
+F 0 "U6" H 925 5025 40  0000 C CNN
+F 1 "EE_Logo" H 925 5085 40  0000 C CNN
+F 2 "" H 925 5175 40  0000 C CNN
+F 3 "" H 925 5175 40  0000 C CNN
+	1    925  5175
+	1    0    0    -1
+$EndComp
+Wire Wire Line
+	10200 5950 10200 5650
 $EndSCHEMATC
